File: pcb_hbridge/project.kicad_sch (KiCad schematic)
At the start: 6 parts, among them IC1 DRV8871DDA, J1 Conn_01x04, J2 Conn_01x04

Commit message: Correct JLCPCB# to LCSC# in BOM
Parts:
- C1: JLCPCB# C473196 -> (none); LCSC# (none) -> C473196
- C2: JLCPCB# C49678 -> (none); LCSC# (none) -> C49678
- IC1: JLCPCB# C1556867 -> (none); LCSC# (none) -> C1556867
- R1: JLCPCB# C319666 -> (none); LCSC# (none) -> C319666
Changed lines of the file:
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@@
-			)
-		)
-		(property "JLCPCB# Alternatives" ""
-			(at 137.16 46.99 0)
-			(effects
-				(font
-					(size 1.27 1.27)
-				)
-				(hide yes)
 			)
 		)
@@
 			)
 		)
-		(property "JLCPCB#" "C1556867"
-			(at 35.56 52.07 0)
-			(effects
-				(font
-					(size 1.27 1.27)
-				)
-				(hide yes)
-			)
-		)
-		(property "JLCPCB# Alternatives" ""
-			(at 35.56 52.07 0)
-			(effects
-				(font
-					(size 1.27 1.27)
-				)
-				(hide yes)
-			)
-		)
 		(property "Manufacturer_Part_Number" "DRV8871DDA"
 			(at 35.56 52.07 0)
@@
 		)
 		(property "digikey#" ""
+			(at 35.56 52.07 0)
+			(effects
+				(font
+					(size 1.27 1.27)
+				)
+				(hide yes)
+			)
+		)
+		(property "LCSC#" "C1556867"
 			(at 35.56 52.07 0)
 			(effects
@@
 			)
 		)
-		(property "JLCPCB#" "C49678"
-			(at 76.2 64.77 0)
-			(effects
-				(font
-					(size 1.27 1.27)
-				)
-				(hide yes)
-			)
-		)
-		(property "JLCPCB# Alternatives" ""
-			(at 76.2 64.77 0)
-			(effects
-				(font
-					(size 1.27 1.27)
-				)
-				(hide yes)
-			)
-		)
 		(property "Manufacturer_Part_Number" "Capacitor, 0.1uF, 50V, 0805 SMD"
 			(at 76.2 64.77 0)
@@
 		)
 		(property "digikey#" ""
+			(at 76.2 64.77 0)
+			(effects
+				(font
+					(size 1.27 1.27)
+				)
+				(hide yes)
+			)
+		)
+		(property "LCSC#" "C49678"
 			(at 76.2 64.77 0)
 			(effects
@@
 			)
 		)
-		(property "JLCPCB#" "C473196"
-			(at 95.25 64.77 0)
-			(effects
-				(font
-					(size 1.27 1.27)
-				)
-				(hide yes)
-			)
-		)
-		(property "JLCPCB# Alternatives" ""
-			(at 95.25 64.77 0)
-			(effects
-				(font
-					(size 1.27 1.27)
-				)
-				(hide yes)
-			)
-		)
 		(property "Manufacturer_Part_Number" "Capacitor, 22.0uF, 63V, D6.3xL7.7 SMD"
 			(at 95.25 64.77 0)
@@
 		)
 		(property "digikey#" ""
+			(at 95.25 64.77 0)
+			(effects
+				(font
+					(size 1.27 1.27)
+				)
+				(hide yes)
+			)
+		)
+		(property "LCSC#" "C473196"
 			(at 95.25 64.77 0)
 			(effects
@@
 			)
 		)
-		(property "JLCPCB# Alternatives" ""
-			(at 137.16 60.96 0)
-			(effects
-				(font
-					(size 1.27 1.27)
-				)
-				(hide yes)
-			)
-		)
 		(property "Manufacturer_Part_Number" ""
 			(at 137.16 60.96 0)
@@
 			)
 		)
-		(property "JLCPCB#" "C319666"
-			(at 31.75 66.04 0)
-			(effects
-				(font
-					(size 1.27 1.27)
-				)
-				(hide yes)
-			)
-		)
-		(property "JLCPCB# Alternatives" ""
-			(at 31.75 66.04 0)
-			(effects
-				(font
-					(size 1.27 1.27)
-				)
-				(hide yes)
-			)
-		)
 		(property "Manufacturer_Part_Number" "Resistor, 30.0kΩ, 1206 SMD"
 			(at 31.75 66.04 0)
@@
 			(at 31.75 66.04 0)
 			(effects
+				(font
+					(size 1.27 1.27)
+				)
+				(hide yes)
+			)
+		)
+		(property "LCSC#" "C319666"
+			(at 31.75 66.04 0)
+			(effects
