File: pcb_main/project.kicad_sch (KiCad schematic)
At the start: 40 parts, among them IC1 SX1509QBIULTRT, J1 Conn_01x04, J10 Conn_01x02, J11 Conn_02x02_Odd_Even, J12 Conn_02x02_Odd_Even, J13 Conn_01x02, J14 Conn_01x04, J15 Conn_01x04, J16 Conn_01x04, J17 Conn_01x04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

Commit message: correct bom columns
Parts:
- J22, J23, J24, J25, J26, J27, J28, J29: Mouser# 538-105313-1103 -> 538-105313-1103

Commit message: Correct JLCPCB# to LCSC# in BOM
Parts:
- C1, C2: JLCPCB# C110251 -> (none); LCSC# (none) -> C110251
- IC1: JLCPCB# C2652294 -> (none); LCSC# (none) -> C2652294
- J10, J13, J9: JLCPCB# C492401 -> (none); LCSC# (none) -> C492401
- J11, J12: JLCPCB# C492419 -> (none); LCSC# (none) -> C492419
- R1, R2, R3, R4: JLCPCB# C60490 -> (none); LCSC# (none) -> C60490
