File: pcb_core/ioexpender.kicad_sch (KiCad schematic)
At the start: 5 parts, among them IC2 SX1509QBIULTRT

Commit message: Correct ECR Warnings
Parts:
- IC2: Arrow Part Number (none) -> SX1509QBIULTRT; Arrow Price/Stock (none) -> https://www.arrow.com/en/products/sx1509qbiultrt/semtech?re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; Mouser Price/Stock (none) -> https://www.mouser.co.uk/ProductDetail/Semtech/SX1509QBIULT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
Changed lines of the file:
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@@
 			)
 		)
-		(property "Description" ""
+		(property "Description" "Voltage Level Shifting GPIO with LED Driver 28-Pin QFN-UT EP T/R"
 			(at 72.39 67.31 0)
 			(effects
@@
 				(hide yes)
 			)
+		)
+		(property "Mouser Price/Stock" "https://www.mouser.co.uk/ProductDetail/Semtech/SX1509QBIULTRT?qs=rBWM4%252BvDhIf3%2FilU3NIYqw%3D%3D"
+			(at 104.14 849.53 0)
+			(effects
+				(font
+					(size 1.27 1.27)
+				)
+				(justify left top)
+				(hide yes)
+			)
+		)
+		(property "Arrow Part Number" "SX1509QBIULTRT"
+			(at 104.14 949.53 0)
+			(effects
+				(font
+					(size 1.27 1.27)
+				)
+				(justify left top)
+				(hide yes)
+			)
+		)
+		(property "Arrow Price/Stock" "https://www.arrow.com/en/products/sx1509qbiultrt/semtech?region=nac"
+			(at 104.14 1049.53 0)
+			(effects
+				(font
+					(size 1.27 1.27)
+				)
+				(justify left top)
+				(hide yes)
+			)

Commit message: Harmonize package sizing of components
Parts:
- C8: footprint Capacitor_SMD:C_0402_1005Metric -> Capacitor_SMD:C_0805_2012Metric_Pad1.18x1.45mm_HandSolder; LCSC# C110251 -> C49678; Manufacturer_Part_Number Capacitor, 0.1uF, 50V, 0402 SMD -> Capacitor, 0.1uF, 50V, 0805 SMD
- C9: footprint Capacitor_SMD:C_0402_1005Metric -> Capacitor_SMD:C_0805_2012Metric_Pad1.18x1.45mm_HandSolder; LCSC# C110251 -> C49678; Manufacturer_Part_Number (none) -> Capacitor, 0.1uF, 50V, 0805 SMD
- R11, R12: footprint Resistor_SMD:R_0402_1005Metric -> Resistor_SMD:R_1206_3216Metric_Pad1.30x1.75mm_HandSolder; LCSC# C60490 -> (none)
Changed lines of the file:
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@@
 			)
 		)
-		(property "Footprint" "Capacitor_SMD:C_0402_1005Metric"
+		(property "Footprint" "Capacitor_SMD:C_0805_2012Metric_Pad1.18x1.45mm_HandSolder"
 			(at 136.8552 85.09 0)
 			(effects
@@
 			)
 		)
-		(property "Description" "Capacitor, 0.1uF, 50V, 0402 SMD"
+		(property "Description" "Capacitor, 0.1uF, 50V, 0805 SMD"
 			(at 135.89 81.28 0)
 			(effects
@@
 			)
 		)
-		(property "Manufacturer_Part_Number" ""
+		(property "Manufacturer_Part_Number" "Capacitor, 0.1uF, 50V, 0805 SMD"
 			(at 135.89 81.28 0)
 			(effects
@@
 			)
 		)
-		(property "LCSC#" "C110251"
+		(property "LCSC#" "C49678"
 			(at 135.89 81.28 0)
 			(effects
@@
 			)
 		)
-		(property "Footprint" "Capacitor_SMD:C_0402_1005Metric"
+		(property "Footprint" "Capacitor_SMD:C_0805_2012Metric_Pad1.18x1.45mm_HandSolder"
 			(at 53.0352 85.09 0)
 			(effects
@@
 			)
 		)
-		(property "Description" "Capacitor, 0.1uF, 50V, 0402 SMD"
+		(property "Description" "Capacitor, 0.1uF, 50V, 0805 SMD"
 			(at 52.07 81.28 0)
 			(effects
@@
 			)
 		)
-		(property "Manufacturer_Part_Number" "Capacitor, 0.1uF, 50V, 0402 SMD"
+		(property "Manufacturer_Part_Number" "Capacitor, 0.1uF, 50V, 0805 SMD"
 			(at 52.07 81.28 0)
 			(effects
@@
 			)
 		)
-		(property "LCSC#" "C110251"
+		(property "LCSC#" "C49678"
 			(at 52.07 81.28 0)
 			(effects
@@
 			)
 		)
-		(property "Footprint" "Resistor_SMD:R_0402_1005Metric"
+		(property "Footprint" "Resistor_SMD:R_1206_3216Metric_Pad1.30x1.75mm_HandSolder"
 			(at 86.868 114.3 90)
 			(effects
@@
 			)
 		)
-		(property "Description" "Resistor, 10.0k, 0402 SMD"
+		(property "Description" "Resistor, 10.0k, 1206 SMD"
 			(at 85.09 114.3 0)
 			(effects
@@
 			)
 		)
-		(property "LCSC#" "C60490"
+		(property "LCSC#" ""
 			(at 85.09 114.3 0)
 			(effects
@@
 			)
 		)
-		(property "Footprint" "Resistor_SMD:R_0402_1005Metric"
+		(property "Footprint" "Resistor_SMD:R_1206_3216Metric_Pad1.30x1.75mm_HandSolder"
 			(at 97.028 33.02 90)
 			(effects
@@
 			)
 		)
-		(property "Description" "Resistor, 10.0k, 0402 SMD"
+		(property "Description" "Resistor, 10.0k, 1206 SMD"
 			(at 95.25 33.02 0)
 			(effects
@@
 			)
 		)
-		(property "LCSC#" "C60490"
+		(property "LCSC#" ""
 			(at 95.25 33.02 0)
 			(effects
