File: pcb_core/ioexpender.kicad_sch (KiCad schematic)
At the start: 5 parts, among them IC2 SX1509QBIULTRT

Commit message: Update BOM
Parts:
- R11, R12: LCSC# (none) -> C17902
Changed lines of the file:
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@@
 			)
 		)
-		(property "LCSC#" ""
+		(property "LCSC#" "C17902"
 			(at 85.09 114.3 0)
 			(effects
@@
 			)
 		)
-		(property "LCSC#" ""
+		(property "LCSC#" "C17902"
 			(at 95.25 33.02 0)
 			(effects

Commit message: Add AISLER bom support and assigned components
Parts:
- C8, C9: AISLER_MPN (none) -> 100.0nF, 0805 SMD
- IC2: AISLER_MPN (none) -> SX1509QBIULTRT
- R11, R12: AISLER_MPN (none) -> 10.0kΩ, 1206 SMD
Changed lines of the file:
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@@
+			)
+		)
+		(property "AISLER_MPN" "100.0nF, 0805 SMD"
+			(at 135.89 81.28 0)
+			(effects
+				(font
+					(size 1.27 1.27)
+				)
+				(hide yes)
 			)
 		)
@@
 			)
 		)
+		(property "AISLER_MPN" "100.0nF, 0805 SMD"
+			(at 52.07 81.28 0)
+			(effects
+				(font
+					(size 1.27 1.27)
+				)
+				(hide yes)
+			)
+		)
 		(pin "2"
 		)
@@
 			)
 		)
+		(property "AISLER_MPN" "10.0kΩ, 1206 SMD "
+			(at 85.09 114.3 0)
+			(effects
+				(font
+					(size 1.27 1.27)
+				)
+				(hide yes)
+			)
+		)
 		(pin "2"
 		)
@@
 			)
 		)
+		(property "AISLER_MPN" "10.0kΩ, 1206 SMD "
+			(at 95.25 33.02 0)
+			(effects
+				(font
+					(size 1.27 1.27)
+				)
+				(hide yes)
+			)
+		)
 		(pin "2"
 		)
@@
 			(at 72.39 67.31 0)
 			(effects
+				(font
+					(size 1.27 1.27)
+				)
+				(hide yes)
+			)
+		)
+		(property "AISLER_MPN" "SX1509QBIULTRT"
+			(at 72.39 67.31 0)
+			(effects

Commit message: Update BOM Mouser
Parts:
- C8, C9: Mouser Part Number (none) -> 80-C0805C104M5R
- R11, R12: Mouser Part Number (none) -> 603-RC1206FR-1010KL
Changed lines of the file:
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@@
+			)
+		)
+		(property "Mouser Part Number" " 80-C0805C104M5R "
+			(at 135.89 81.28 0)
+			(effects
+				(font
+					(size 1.27 1.27)
+				)
+				(hide yes)
+			)
+		)
+		(property "Mouser# Alt1" ""
+			(at 135.89 81.28 0)
+			(effects
+				(font
+					(size 1.27 1.27)
+				)
+				(hide yes)
 			)
 		)
@@
 			)
 		)
+		(property "Mouser Part Number" " 80-C0805C104M5R "
+			(at 52.07 81.28 0)
+			(effects
+				(font
+					(size 1.27 1.27)
+				)
+				(hide yes)
+			)
+		)
+		(property "Mouser# Alt1" ""
+			(at 52.07 81.28 0)
+			(effects
+				(font
+					(size 1.27 1.27)
+				)
+				(hide yes)
+			)
+		)
 		(pin "2"
 		)
@@
 			)
 		)
+		(property "Mouser Part Number" "603-RC1206FR-1010KL"
+			(at 85.09 114.3 0)
+			(effects
+				(font
+					(size 1.27 1.27)
+				)
+				(hide yes)
+			)
+		)
+		(property "Mouser# Alt1" ""
+			(at 85.09 114.3 0)
+			(effects
+				(font
+					(size 1.27 1.27)
+				)
+				(hide yes)
+			)
+		)
 		(pin "2"
 		)
@@
 			)
 		)
+		(property "Mouser Part Number" "603-RC1206FR-1010KL"
+			(at 95.25 33.02 0)
+			(effects
+				(font
+					(size 1.27 1.27)
+				)
+				(hide yes)
+			)
+		)
+		(property "Mouser# Alt1" ""
+			(at 95.25 33.02 0)
+			(effects
+				(font
+					(size 1.27 1.27)
+				)
+				(hide yes)
+			)
+		)
 		(pin "2"
 		)
@@
 			(at 72.39 67.31 0)
 			(effects
+				(font
+					(size 1.27 1.27)
+				)
+				(hide yes)
+			)
+		)
+		(property "Mouser# Alt1" ""
+			(at 72.39 67.31 0)
+			(effects

Commit message: New package version of model train controller
Parts:
- removed C8, C9: 0.1uF, Capacitor_SMD:C_0805_2012Metric_Pad1.18x1.45mm_HandSolder, symbol Device:C
- removed IC2: SX1509QBIULTRT, library:QFN40P400X400X60-29N-D, symbol SX1509QBIULTRT:SX1509QBIULTRT
- removed R11, R12: 10k, Resistor_SMD:R_1206_3216Metric_Pad1.30x1.75mm_HandSolder, symbol Device:R
Connections:
- no-connect marks 1 -> 0
