File: pcb_core/project.kicad_sch (KiCad schematic)
At the start: 53 parts, among them IC4 TCA9548APWR, J1 Conn_01x02, J19 Conn_02x02_Counter_Clockwise, J2 1725656, J20 PCBConnector, J21 PCBConnector, J22 PCBConnector, J23 PCBConnector, J25 PCBConnector, J27 PCBConnector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

Commit message: Add variants for Master and Slave
Parts:
- C1, C2, C3, C4, C5, R2, S1, S2: config (none) -> +MasterESP32S3
- C41, C42, C45, Q1, U2: config (none) -> -Slave
- J1, R14, R15: config (none) -> +MasterESP32S3,+MasterESP32Devkit
- U1, U3: config (none) -> +MasterESP32Devkit

Commit message: Convert 'config' to 'Config'
Parts:
- C1, C2, C3, C4, C5, R2, S1, S2: Config (none) -> +MasterESP32S3; config +MasterESP32S3 -> (none)
- C41, C42, C45, Q1, U2: Config (none) -> -Slave; config -Slave -> (none)
- J1, R14, R15: Config (none) -> +MasterESP32S3,+MasterESP32Devkit; config +MasterESP32S3,+MasterESP32Devkit -> (none)
- U1, U3: Config (none) -> +MasterESP32Devkit; config +MasterESP32Devkit -> (none)
Changed lines of the file:
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@@
 			)
 		)
-		(property "config" ""
+		(property "Config" ""
 			(at 447.04 389.89 0)
 			(effects
@@
 			)
 		)
-		(property "config" ""
+		(property "Config" ""
 			(at 447.04 374.65 0)
 			(effects
@@
 			)
 		)
-		(property "config" ""
+		(property "Config" ""
 			(at 114.3 356.87 0)
 			(effects
@@
 			)
 		)
-		(property "config" ""
+		(property "Config" ""
 			(at 414.02 387.35 0)
 			(effects
@@
 			)
 		)
-		(property "config" "+MasterESP32S3,+MasterESP32Devkit"
+		(property "Config" "+MasterESP32S3,+MasterESP32Devkit"
 			(at 176.53 121.92 0)
 			(effects
@@
 			)
 		)
-		(property "config" ""
+		(property "Config" ""
 			(at 100.33 379.73 0)
 			(effects
@@
 			)
 		)
-		(property "config" "-Slave"
+		(property "Config" "-Slave"
 			(at 386.08 361.95 0)
 			(effects
@@
 			)
 		)
-		(property "config" ""
+		(property "Config" ""
 			(at 55.88 228.6 0)
 			(effects
@@
 			)
 		)
-		(property "config" ""
+		(property "Config" ""
 			(at 22.86 264.16 0)
 			(effects
@@
 			)
 		)
-		(property "config" ""
+		(property "Config" ""
 			(at 34.29 241.3 0)
 			(effects
@@
 			)
 		)
-		(property "config" "-Slave"
+		(property "Config" "-Slave"
 			(at 143.51 365.76 0)
 			(effects
@@
 			)
 		)
-		(property "config" ""
+		(property "Config" ""
 			(at 365.76 387.35 0)
 			(effects
@@
 			)
 		)
-		(property "config" "+MasterESP32S3"
+		(property "Config" "+MasterESP32S3"
 			(at 214.63 22.86 0)
 			(effects
@@
 			)
 		)
-		(property "config" ""
+		(property "Config" ""
 			(at 114.3 373.38 0)
 			(effects
@@
 			)
 		)
-		(property "config" ""
+		(property "Config" ""
 			(at 346.71 364.49 0)
 			(effects
@@
 			)
 		)
-		(property "config" ""
+		(property "Config" ""
 			(at 100.33 388.62 0)
 			(effects
@@
 			)
 		)
-		(property "config" ""
+		(property "Config" ""
 			(at 396.24 344.17 0)
 			(effects
@@
 			)
 		)
-		(property "config" ""
+		(property "Config" ""
 			(at 85.09 356.87 0)
 			(effects
@@
 			)
 		)
-		(property "config" ""
+		(property "Config" ""
 			(at 109.22 233.68 0)
 			(effects
@@
 			)
 		)
-		(property "config" "+MasterESP32Devkit"
+		(property "Config" "+MasterESP32Devkit"
 			(at 120.65 81.28 0)
 			(effects
@@
 			)
 		)
-		(property "config" "+MasterESP32Devkit"
+		(property "Config" "+MasterESP32Devkit"
 			(at 335.28 97.79 0)
 			(effects
@@
 			)
 		)
-		(property "config" "+MasterESP32S3"
+		(property "Config" "+MasterESP32S3"
 			(at 238.76 67.31 0)
 			(effects
@@
 			)
 		)
-		(property "config" ""
+		(property "Config" ""
 			(at 414.02 379.73 0)
 			(effects
@@
 			)
 		)
-		(property "config" ""
+		(property "Config" ""
 			(at 203.2 107.95 0)
 			(effects
@@
 			)
 		)
-		(property "config" ""
+		(property "Config" ""
 			(at 447.04 369.57 0)
 			(effects
@@
 			)
 		)
-		(property "config" ""
+		(property "Config" ""
 			(at 447.04 400.05 0)
 			(effects
@@
 			)
 		)
-		(property "config" ""
+		(property "Config" ""
 			(at 114.3 383.54 0)
 			(effects
@@
 			)
 		)
-		(property "config" ""
+		(property "Config" ""
 			(at 113.03 25.4 0)
 			(effects
@@
 			)
 		)
-		(property "config" "-Slave"
+		(property "Config" "-Slave"
 			(at 382.27 337.82 0)
 			(effects
@@
 			)
 		)
-		(property "config" ""
+		(property "Config" ""
 			(at 30.48 264.16 0)
 			(effects
@@
 			)
 		)
-		(property "config" "+MasterESP32S3,+MasterESP32Devkit"
+		(property "Config" "+MasterESP32S3,+MasterESP32Devkit"
 			(at 176.53 109.22 0)
 			(effects
@@
 			)
 		)
-		(property "config" ""
+		(property "Config" ""
 			(at 38.1 264.16 0)
 			(effects
@@
 			)
 		)
-		(property "config" "+MasterESP32S3"
+		(property "Config" "+MasterESP32S3"
 			(at 238.76 80.01 0)
 			(effects
@@
 			)
 		)
-		(property "config" ""
+		(property "Config" ""
 			(at 100.33 369.57 0)
 			(effects
@@
 			)
 		)
-		(property "config" ""
+		(property "Config" ""
 			(at 172.72 382.27 0)
 			(effects
@@
 			)
 		)
-		(property "config" ""
+		(property "Config" ""
 			(at 447.04 405.13 0)
 			(effects
@@
 			)
 		)
-		(property "config" ""
+		(property "Config" ""
 			(at 203.2 123.19 0)
 			(effects
@@
 			)
 		)
-		(property "config" "+MasterESP32S3"
+		(property "Config" "+MasterESP32S3"
 			(at 269.24 21.59 0)
 			(effects
@@
 			)
 		)
-		(property "config" ""
+		(property "Config" ""
 			(at 447.04 384.81 0)
 			(effects
@@
 			)
 		)
-		(property "config" "+MasterESP32S3,+MasterESP32Devkit"
+		(property "Config" "+MasterESP32S3,+MasterESP32Devkit"
 			(at 353.06 29.21 0)
 			(effects
@@
 			)
 		)
-		(property "config" ""
+		(property "Config" ""
 			(at 172.72 373.38 0)
 			(effects
@@
 			)
 		)
-		(property "config" "+MasterESP32S3"
-			(at 284.48 38.1 90)
+		(property "Config" "+MasterESP32S3"
+			(at 284.48 38.1 0)
 			(effects
 				(font
@@
 			)
 		)
-		(property "config" "-Slave"
+		(property "Config" "-Slave"
 			(at 140.97 344.17 0)
 			(effects
@@
 			)
 		)
-		(property "config" "+MasterESP32S3"
+		(property "Config" "+MasterESP32S3"
 			(at 102.87 31.75 0)
 			(effects
@@
 			)
 		)
-		(property "config" "+MasterESP32S3"
-			(at 229.87 38.1 90)
+		(property "Config" "+MasterESP32S3"
+			(at 229.87 38.1 0)
 			(effects
 				(font
@@
 			)
 		)
-		(property "config" "-Slave"
+		(property "Config" "-Slave"
 			(at 162.56 367.03 0)
 			(effects
@@
 			)
 		)
-		(property "config" ""
+		(property "Config" ""
 			(at 447.04 379.73 0)
 			(effects
@@
 			)
 		)
-		(property "config" ""
+		(property "Config" ""
 			(at 45.72 264.16 0)
 			(effects
@@
 			)
 		)
-		(property "config" ""
+		(property "Config" ""
 			(at 346.71 345.44 0)
 			(effects
@@
 			)
 		)
-		(property "config" ""
+		(property "Config" ""
 			(at 414.02 397.51 0)
 			(effects
@@
 			)
 		)
-		(property "config" ""
+		(property "Config" ""
 			(at 447.04 394.97 0)
 			(effects
@@
 			)
 		)
-		(property "config" ""
+		(property "Config" ""
 			(at 41.91 205.74 0)
 			(effects
@@
 			)
 		)
-		(property "config" "+MasterESP32S3"
+		(property "Config" "+MasterESP32S3"
 			(at 91.44 31.75 0)
 			(effects

Commit message: Correct variant setting for components
Parts:
- D1, D3, D4, PS1, R4, R5, R6, R7: Config (none) -> -Slave
- R14, R15: Config +MasterESP32S3,+MasterESP32Devkit -> (none)
- U1: Config +MasterESP32Devkit -> +MasterESP32S3
Changed lines of the file:
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@@
 			)
 		)
-		(property "Config" ""
+		(property "Config" "-Slave"
 			(at 114.3 356.87 0)
 			(effects
@@
 			)
 		)
-		(property "Config" "+MasterESP32S3,+MasterESP32Devkit"
+		(property "Config" ""
 			(at 176.53 121.92 0)
 			(effects
@@
 			)
 		)
-		(property "Config" ""
+		(property "Config" "-Slave"
 			(at 100.33 379.73 0)
 			(effects
@@
 			)
 		)
-		(property "Config" ""
+		(property "Config" "-Slave"
 			(at 114.3 373.38 0)
 			(effects
@@
 			)
 		)
-		(property "Config" ""
+		(property "Config" "-Slave"
 			(at 100.33 388.62 0)
 			(effects
@@
 			)
 		)
-		(property "Config" ""
+		(property "Config" "-Slave"
 			(at 396.24 344.17 0)
 			(effects
@@
 			)
 		)
-		(property "Config" ""
+		(property "Config" "-Slave"
 			(at 85.09 356.87 0)
 			(effects
@@
 			)
 		)
-		(property "Config" "+MasterESP32Devkit"
+		(property "Config" "+MasterESP32S3"
 			(at 120.65 81.28 0)
 			(effects
@@
 			)
 		)
-		(property "Config" ""
+		(property "Config" "-Slave"
 			(at 114.3 383.54 0)
 			(effects
@@
 			)
 		)
-		(property "Config" "+MasterESP32S3,+MasterESP32Devkit"
+		(property "Config" ""
 			(at 176.53 109.22 0)
 			(effects
@@
 			)
 		)
-		(property "Config" ""
+		(property "Config" "-Slave"
 			(at 100.33 369.57 0)
 			(effects

Commit message: Move location of power line led and set LCSC-IDs
Parts:
- added R1, R22: 1.1k, Resistor_SMD:R_1206_3216Metric_Pad1.30x1.75mm_HandSolder, symbol Device:R
- D2: LCSC# (none) -> C2980185
- D3: LCSC# (none) -> C84270
- R3: Config (none) -> +MasterESP32S3
- U3: LCSC# (none) -> C571180
Connections:
- net at D4.1 (K): now also R22.1; no longer D3.2 (A)
- net at D2.2 (A): now also R1.2; no longer D5.1 (K)
- new net: D3.2 (A), R22.2
- new net: D5.1 (K), R1.1
Other:
- moved on the sheet: D2, D3
Changed lines of the file:
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@@
 	(wire
 		(pts
-			(xy 172.72 386.08) (xy 172.72 388.62)
+			(xy 172.72 396.24) (xy 172.72 398.78)
 		)
 		(stroke
@@
 	(wire
 		(pts
-			(xy 172.72 377.19) (xy 172.72 378.46)
+			(xy 172.72 377.19) (xy 172.72 379.73)
 		)
 		(stroke
@@
 	(wire
 		(pts
+			(xy 172.72 387.35) (xy 172.72 388.62)
+		)
+		(stroke
+			(width 0)
+			(type default)
+		)
+	)
+	(wire
+		(pts
 			(xy 368.3 67.31) (xy 370.84 67.31)
 		)
@@
 	(wire
 		(pts
+			(xy 100.33 392.43) (xy 100.33 393.7)
+		)
+		(stroke
+			(width 0)
+			(type default)
+		)
+	)
+	(wire
+		(pts
 			(xy 492.76 337.82) (xy 495.3 337.82)
 		)
@@
 	(wire
 		(pts
-			(xy 157.48 398.78) (xy 157.48 363.22)
+			(xy 157.48 403.86) (xy 157.48 363.22)
 		)
 		(stroke
@@
 	(wire
 		(pts
-			(xy 100.33 392.43) (xy 100.33 398.78)
+			(xy 100.33 401.32) (xy 100.33 403.86)
 		)
 		(stroke
@@
 	(wire
 		(pts
-			(xy 100.33 398.78) (xy 157.48 398.78)
+			(xy 100.33 403.86) (xy 157.48 403.86)
 		)
 		(stroke
@@
 	(global_label "GNDA"
 		(shape passive)
-		(at 172.72 388.62 270)
+		(at 172.72 398.78 270)
 		(fields_autoplaced yes)
 		(effects
@@
 		)
 		(property "Intersheetrefs" "${INTERSHEET_REFS}"
-			(at 172.72 395.453 90)
+			(at 172.72 405.613 90)
 			(effects
 				(font
@@
 	(symbol
 		(lib_id "Device:LED")
-		(at 100.33 388.62 90)
+		(at 100.33 397.51 90)
 		(unit 1)
 		(exclude_from_sim no)
@@
 		(fields_autoplaced yes)
 		(property "Reference" "D3"
-			(at 104.14 388.9374 90)
+			(at 104.14 397.8274 90)
 			(effects
 				(font
@@
 		)
 		(property "Value" "RED LED"
-			(at 104.14 391.4774 90)
+			(at 104.14 400.3674 90)
 			(effects
 				(font
@@
 		)
 		(property "Footprint" "LED_SMD:LED_1206_3216Metric_Pad1.42x1.75mm_HandSolder"
-			(at 100.33 388.62 0)
+			(at 100.33 397.51 0)
 			(effects
 				(font
@@
 		)
 		(property "Datasheet" "~"
-			(at 100.33 388.62 0)
+			(at 100.33 397.51 0)
 			(effects
 				(font
@@
 		)
 		(property "Description" "Light emitting diode"
-			(at 100.33 388.62 0)
+			(at 100.33 397.51 0)
 			(effects
 				(font
@@
 		)
 		(property "Config" "-Slave"
-			(at 100.33 388.62 0)
+			(at 100.33 397.51 0)
+			(effects
+				(font
+					(size 1.27 1.27)
+				)
+				(hide yes)
+			)
+		)
+		(property "LCSC#" "C84270"
+			(at 100.33 397.51 0)
 			(effects
 				(font
@@
 			)
 		)
+		(property "LCSC#" "C571180"
+			(at 335.28 97.79 0)
+			(effects
+				(font
+					(size 1.27 1.27)
+				)
+				(hide yes)
+			)
+		)
 		(pin "3"
 		)
@@
 			)
 		)
-		(property "Config" ""
+		(property "Config" "+MasterESP32S3"
 			(at 113.03 25.4 0)
 			(effects
@@
 	(symbol
 		(lib_id "Device:R")
+		(at 100.33 388.62 0)
+		(unit 1)
+		(exclude_from_sim no)
+		(in_bom yes)
+		(on_board yes)
+		(dnp no)
+		(fields_autoplaced yes)
+		(property "Reference" "R22"
+			(at 102.87 387.3499 0)
+			(effects
+				(font
+					(size 1.27 1.27)
+				)
+				(justify left)
+			)
+		)
+		(property "Value" "1.1k"
+			(at 102.87 389.8899 0)
+			(effects
+				(font
+					(size 1.27 1.27)
+				)
+				(justify left)
+			)
+		)
+		(property "Footprint" "Resistor_SMD:R_1206_3216Metric_Pad1.30x1.75mm_HandSolder"
+			(at 98.552 388.62 90)
+			(effects
+				(font
+					(size 1.27 1.27)
+				)
+				(hide yes)
+			)
+		)
+		(property "Datasheet" "~"
+			(at 100.33 388.62 0)
+			(effects
+				(font
+					(size 1.27 1.27)
+				)
+				(hide yes)
+			)
+		)
+		(property "Description" "Resistor, 1.1k, 1206 SMD"
+			(at 100.33 388.62 0)
+			(effects
+				(font
+					(size 1.27 1.27)
+				)
+				(hide yes)
+			)
+		)
+		(property "LCSC#" " C2933580"
+			(at 100.33 388.62 0)
+			(effects
+				(font
+					(size 1.27 1.27)
+				)
+				(hide yes)
+			)
+		)
+		(pin "1"
+		)
+		(pin "2"
+		)
+		(instances
+			(project "project"
+				(path "/97ee99f6-6664-45d1-b5d6-247aaf34e934"
+					(reference "R22")
+					(unit 1)
+				)
+			)
+		)
+	)
+	(symbol
+		(lib_id "Device:R")
 		(at 38.1 264.16 180)
 		(unit 1)
@@
 	(symbol
 		(lib_id "Device:LED")
-		(at 172.72 382.27 90)
+		(at 172.72 392.43 90)
 		(unit 1)
 		(exclude_from_sim no)
@@
 		(fields_autoplaced yes)
 		(property "Reference" "D2"
-			(at 176.53 382.5874 90)
+			(at 176.53 392.7474 90)
 			(effects
 				(font
@@
 		)
 		(property "Value" "GREEN LED"
-			(at 176.53 385.1274 90)
+			(at 176.53 395.2874 90)
 			(effects
 				(font
@@
 		)
 		(property "Footprint" "LED_SMD:LED_1206_3216Metric_Pad1.42x1.75mm_HandSolder"
-			(at 172.72 382.27 0)
+			(at 172.72 392.43 0)
 			(effects
 				(font
@@
 		)
 		(property "Datasheet" "~"
-			(at 172.72 382.27 0)
+			(at 172.72 392.43 0)
 			(effects
 				(font
@@
 		)
 		(property "Description" "Light emitting diode"
-			(at 172.72 382.27 0)
+			(at 172.72 392.43 0)
 			(effects
 				(font
@@
 		)
 		(property "Config" ""
-			(at 172.72 382.27 0)
+			(at 172.72 392.43 0)
+			(effects
+				(font
+					(size 1.27 1.27)
+				)
+				(hide yes)
+			)
+		)
+		(property "LCSC#" "C2980185"
+			(at 172.72 392.43 0)
 			(effects
 				(font
@@
 					(unit 1)
 				)
+			)
+		)
+	)
+	(symbol
+		(lib_id "Device:R")
+		(at 172.72 383.54 0)
+		(unit 1)
+		(exclude_from_sim no)
+		(in_bom yes)
+		(on_board yes)
+		(dnp no)
+		(fields_autoplaced yes)
+		(property "Reference" "R1"
+			(at 175.26 382.2699 0)
+			(effects
+				(font
+					(size 1.27 1.27)
+				)
+				(justify left)
+			)
+		)
+		(property "Value" "1.1k"
+			(at 175.26 384.8099 0)
+			(effects
+				(font
+					(size 1.27 1.27)
+				)
+				(justify left)
+			)
+		)
+		(property "Footprint" "Resistor_SMD:R_1206_3216Metric_Pad1.30x1.75mm_HandSolder"
+			(at 170.942 383.54 90)
+			(effects
+				(font
+					(size 1.27 1.27)
+				)
+				(hide yes)
+			)
+		)
+		(property "Datasheet" "~"
+			(at 172.72 383.54 0)
+			(effects
+				(font
+					(size 1.27 1.27)
+				)
+				(hide yes)
+			)
+		)
+		(property "Description" "Resistor, 1.1k, 1206 SMD"
+			(at 172.72 383.54 0)
+			(effects
+				(font
+					(size 1.27 1.27)
+				)
+				(hide yes)
+			)
+		)
+		(property "LCSC#" " C2933580"
+			(at 172.72 383.54 0)
+			(effects
+				(font
+					(size 1.27 1.27)
+				)
+				(hide yes)
+			)
+		)
+		(pin "1"
+		)
+		(pin "2"
+		)
+		(instances
+			(project "project"
+				(path "/97ee99f6-6664-45d1-b5d6-247aaf34e934"
+					(reference "R1")
+					(unit 1)
+				)

Commit message: Correct variant setting for components
Parts:
- R22: Config (none) -> -Slave
Changed lines of the file:
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@@
+			)
+		)
+		(property "Config" "-Slave"
+			(at 100.33 388.62 0)
+			(effects
+				(font
+					(size 1.27 1.27)
+				)
+				(hide yes)
 			)
 		)
@@
 			(at 172.72 383.54 0)
 			(effects
+				(font
+					(size 1.27 1.27)
+				)
+				(hide yes)
+			)
+		)
+		(property "Config" ""
+			(at 172.72 383.54 0)
+			(effects

Commit message: Change master,slave to primary and sub node
Parts:
- C1, C2, C3, C4, C5, R2, R3, S1, S2, U1: Config +MasterESP32S3 -> +PrimaryNodeESP32S3
- C41, C42, C45, D1, D3, D4, PS1, Q1, R22, R4, R5, R6, R7, U2: Config -Slave -> -SubNode
- J1: Config +MasterESP32S3,+MasterESP32Devkit -> +PrimaryNodeESP32S3,+PrimaryNodeESP32Devkit
- U3: Config +MasterESP32Devkit -> +PrimaryNodeESP32Devkit
Changed lines of the file:
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@@
 			)
 		)
-		(property "Config" "-Slave"
+		(property "Config" "-SubNode "
 			(at 114.3 356.87 0)
 			(effects
@@
 			)
 		)
-		(property "Config" "-Slave"
+		(property "Config" "-SubNode"
 			(at 100.33 379.73 0)
 			(effects
@@
 			)
 		)
-		(property "Config" "-Slave"
+		(property "Config" "-SubNode"
 			(at 386.08 361.95 0)
 			(effects
@@
 			)
 		)
-		(property "Config" "-Slave"
+		(property "Config" "-SubNode "
 			(at 143.51 365.76 0)
 			(effects
@@
 			)
 		)
-		(property "Config" "+MasterESP32S3"
+		(property "Config" "+PrimaryNodeESP32S3"
 			(at 214.63 22.86 0)
 			(effects
@@
 			)
 		)
-		(property "Config" "-Slave"
+		(property "Config" "-SubNode "
 			(at 114.3 373.38 0)
 			(effects
@@
 			)
 		)
-		(property "Config" "-Slave"
+		(property "Config" "-SubNode"
 			(at 100.33 397.51 0)
 			(effects
@@
 			)
 		)
-		(property "Config" "-Slave"
+		(property "Config" "-SubNode "
 			(at 396.24 344.17 0)
 			(effects
@@
 			)
 		)
-		(property "Config" "-Slave"
+		(property "Config" "-SubNode "
 			(at 85.09 356.87 0)
 			(effects
@@
 			)
 		)
-		(property "Config" "+MasterESP32S3"
+		(property "Config" "+PrimaryNodeESP32S3"
 			(at 120.65 81.28 0)
 			(effects
@@
 			)
 		)
-		(property "Config" "+MasterESP32Devkit"
+		(property "Config" "+PrimaryNodeESP32Devkit"
 			(at 335.28 97.79 0)
 			(effects
@@
 			)
 		)
-		(property "Config" "+MasterESP32S3"
+		(property "Config" "+PrimaryNodeESP32S3"
 			(at 238.76 67.31 0)
 			(effects
@@
 			)
 		)
-		(property "Config" "-Slave"
+		(property "Config" "-SubNode "
 			(at 114.3 383.54 0)
 			(effects
@@
 			)
 		)
-		(property "Config" "+MasterESP32S3"
+		(property "Config" "+PrimaryNodeESP32S3"
 			(at 113.03 25.4 0)
 			(effects
@@
 			)
 		)
-		(property "Config" "-Slave"
+		(property "Config" "-SubNode"
 			(at 382.27 337.82 0)
 			(effects
@@
 			)
 		)
-		(property "Config" "-Slave"
+		(property "Config" "-SubNode "
 			(at 100.33 388.62 0)
 			(effects
@@
 			)
 		)
-		(property "Config" "+MasterESP32S3"
+		(property "Config" "+PrimaryNodeESP32S3"
 			(at 238.76 80.01 0)
 			(effects
@@
 			)
 		)
-		(property "Config" "-Slave"
+		(property "Config" "-SubNode"
 			(at 100.33 369.57 0)
 			(effects
@@
 			)
 		)
-		(property "Config" "+MasterESP32S3"
+		(property "Config" "+PrimaryNodeESP32S3"
 			(at 269.24 21.59 0)
 			(effects
@@
 			)
 		)
-		(property "Config" "+MasterESP32S3,+MasterESP32Devkit"
+		(property "Config" "+PrimaryNodeESP32S3,+PrimaryNodeESP32Devkit"
 			(at 353.06 29.21 0)
 			(effects
@@
 			)
 		)
-		(property "Config" "+MasterESP32S3"
+		(property "Config" "+PrimaryNodeESP32S3"
 			(at 284.48 38.1 0)
 			(effects
@@
 			)
 		)
-		(property "Config" "-Slave"
+		(property "Config" "-SubNode "
 			(at 140.97 344.17 0)
 			(effects
@@
 			)
 		)
-		(property "Config" "+MasterESP32S3"
+		(property "Config" "+PrimaryNodeESP32S3"
 			(at 102.87 31.75 0)
 			(effects
@@
 			)
 		)
-		(property "Config" "+MasterESP32S3"
+		(property "Config" "+PrimaryNodeESP32S3"
 			(at 229.87 38.1 0)
 			(effects
@@
 			)
 		)
-		(property "Config" "-Slave"
+		(property "Config" "-SubNode"
 			(at 162.56 367.03 0)
 			(effects
@@
 			)
 		)
-		(property "Config" "+MasterESP32S3"
+		(property "Config" "+PrimaryNodeESP32S3"
 			(at 91.44 31.75 0)
 			(effects

Commit message: Add LED for 3.3V power line
Parts:
- added D6: GREEN LED, LED_SMD:LED_1206_3216Metric_Pad1.42x1.75mm_HandSolder, symbol Device:LED
- added R23: 56, Resistor_SMD:R_1206_3216Metric_Pad1.30x1.75mm_HandSolder, symbol Device:R
Connections:
- net GNDD: now also D6.1 (K)
- net VCC_3V3: now also R23.1
- new net: D6.2 (A), R23.2

Commit message: Update BOM
Parts:
- removed R1, R22: 1.1k, Resistor_SMD:R_1206_3216Metric_Pad1.30x1.75mm_HandSolder, symbol Device:R
- C42: LCSC# C5266037 -> C267471
- D2, D6: LCSC# C2980185 -> C5336737; LCSC# Alt1 (none) -> C99881; Manufacturer_Name (none) -> ROHM Semiconductor; Manufacturer_Part_Number (none) -> SML-012P8TT86; Mouser Part Number (none) -> 755-SML-012P8TT86
- D3: LCSC# C84270 -> C6229209; LCSC# Alt1 (none) -> C84270; Manufacturer_Name (none) -> ROHM Semiconductor; Manufacturer_Part_Number (none) -> SML-012V8TT86; Mouser Part Number (none) -> 755-SML-012V8TT86
- R6: LCSC# C5126164 -> C488644
Connections:
- net at D4.1 (K): now also D3.2 (A)
- net at D2.2 (A): now also D5.1 (K)
Other:
- moved on the sheet: D2, D3
