File: pcb_core/output_connector.kicad_sch (KiCad schematic)
At the start: 5 parts, among them IC1 DRV8871DDA, J3 1053131103

Commit message: New package version of model train controller
Parts:
- renumbered C6 to C21, C7 to C22, IC1 to IC9, J3 to J9, R8 to R33
Other:
- title: Model Train Controller - OutputConnector -> Model Train Controller - Base
