File: pcb_esp32dev/project.kicad_pcb (KiCad board)
At the start: 2 copper layers, 31 x 73.7 mm, 27 parts, among them J1 Conn_01x01, J10 Conn_01x01, J11 Conn_01x01, J12 Conn_01x01, J13 Conn_01x01, J14 Conn_01x01, J15 Conn_01x01, J16 Conn_01x01, J17 Conn_01x01, J18 Conn_01x01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

Commit message: Correct ESP32Dev PCB panelize
Parts:
- moved T7 0.25 mm to (91.4, 47.0)
- moved T8 0.25 mm to (73.2, 47.0)
Changed lines of the file:
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@@
 		(descr "A symbol representing annotation for tab placement")
 		(property "Reference" "T4"
-			(at 0 -2 360)
+			(at 0 -2 0)
 			(layer "F.SilkS")
 			(hide yes)
@@
 		)
 		(property "Value" "Tab"
-			(at -2.75 -1 360)
+			(at -2.75 -1 0)
 			(layer "Dwgs.User")
 			(effects
@@
 		)
 		(property "Footprint" "PCM_kikit:Tab"
-			(at 0 0 360)
+			(at 0 0 0)
 			(layer "F.Fab")
 			(hide yes)
@@
 		)
 		(property "Datasheet" ""
-			(at 0 0 360)
+			(at 0 0 0)
 			(layer "F.Fab")
 			(hide yes)
@@
 		)
 		(property "Description" "KiKit tab annotations"
-			(at 0 0 360)
+			(at 0 0 0)
 			(layer "F.Fab")
 			(hide yes)
@@
 	(footprint "PCM_kikit:Tab"
 		(layer "F.Cu")
-		(at 73.152 46.736)
+		(at 73.152 46.99)
 		(descr "A symbol representing annotation for tab placement")
 		(property "Reference" "T8"
@@
 		)
 		(fp_text user "KIKIT: width: 3mm"
-			(at -5.5 0 360)
+			(at -5.5 0 0)
 			(layer "Dwgs.User")
 			(effects
@@
 		(descr "A symbol representing annotation for tab placement")
 		(property "Reference" "T3"
-			(at 0 -2 360)
+			(at 0 -2 0)
 			(layer "F.SilkS")
 			(hide yes)
@@
 		)
 		(property "Value" "Tab"
-			(at -2.75 -1 360)
+			(at -2.75 -1 0)
 			(layer "Dwgs.User")
 			(effects
@@
 		)
 		(property "Footprint" "PCM_kikit:Tab"
-			(at 0 0 360)
+			(at 0 0 0)
 			(layer "F.Fab")
 			(hide yes)
@@
 		)
 		(property "Datasheet" ""
-			(at 0 0 360)
+			(at 0 0 0)
 			(layer "F.Fab")
 			(hide yes)
@@
 		)
 		(property "Description" "KiKit tab annotations"
-			(at 0 0 360)
+			(at 0 0 0)
 			(layer "F.Fab")
 			(hide yes)
@@
 	(footprint "PCM_kikit:Tab"
 		(layer "F.Cu")
-		(at 91.44 46.736 180)
+		(at 91.44 46.99 180)
 		(descr "A symbol representing annotation for tab placement")
 		(property "Reference" "T7"
-			(at 0 -2 360)
+			(at 0 -2 0)
 			(layer "F.SilkS")
 			(hide yes)
@@
 		)
 		(property "Value" "Tab"
-			(at -2.75 -1 360)
+			(at -2.75 -1 0)
 			(layer "Dwgs.User")
 			(effects
@@
 		)
 		(property "Footprint" "PCM_kikit:Tab"
-			(at 0 0 360)
+			(at 0 0 0)
 			(layer "F.Fab")
 			(hide yes)
@@
 		)
 		(property "Datasheet" ""
-			(at 0 0 360)
+			(at 0 0 0)
 			(layer "F.Fab")
 			(hide yes)
@@
 		)
 		(property "Description" "KiKit tab annotations"
-			(at 0 0 360)
+			(at 0 0 0)
 			(layer "F.Fab")
 			(hide yes)
@@
 		)
 		(fp_text user "KIKIT: width: 3mm"
-			(at -5.5 0 360)
-			(layer "Dwgs.User")
-			(effects
+			(at -5.5 0 0)
+			(layer "Dwgs.User")
+			(effects
