File: pcb_vpdummy/project.kicad_pcb (KiCad board)
At the start: 2 copper layers, 18 x 16 mm, 16 parts, among them J1 Conn_01x01, J10 Conn_01x01, J11 Conn_01x01, J12 Conn_01x01, J2 Conn_01x01, J3 Conn_01x01, J4 Conn_01x01, J5 Conn_01x01, J6 Conn_01x01, J7 Conn_01x01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

Commit message: Correct ESP32Dev PCB panelize
Parts:
- moved T1 0.51 mm to (78.0, 39.6)
- moved T2 0.51 mm to (92.5, 39.6)
- moved T3 0.51 mm to (78.0, 56.1)
- moved T4 0.51 mm to (92.5, 56.2)
Changed lines of the file:
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@@
 	(footprint "PCM_kikit:Tab"
 		(layer "F.Cu")
-		(at 92.964 39.624 -90)
+		(at 92.456 39.624 -90)
 		(descr "A symbol representing annotation for tab placement")
 		(property "Reference" "T2"
@@
 		)
 		(fp_text user "KIKIT: width: 3mm"
-			(at -5.5 0 360)
+			(at -5.5 0 0)
 			(layer "Dwgs.User")
 			(effects
@@
 	(footprint "PCM_kikit:Tab"
 		(layer "F.Cu")
-		(at 77.47 39.624 -90)
+		(at 77.978 39.624 -90)
 		(descr "A symbol representing annotation for tab placement")
 		(property "Reference" "T1"
@@
 		)
 		(fp_text user "KIKIT: width: 3mm"
-			(at -5.5 0 360)
+			(at -5.5 0 0)
 			(layer "Dwgs.User")
 			(effects
@@
 	(footprint "PCM_kikit:Tab"
 		(layer "F.Cu")
-		(at 77.47 56.134 90)
+		(at 77.978 56.134 90)
 		(descr "A symbol representing annotation for tab placement")
 		(property "Reference" "T3"
@@
 		)
 		(fp_text user "KIKIT: width: 3mm"
-			(at -5.5 0 360)
+			(at -5.5 0 0)
 			(layer "Dwgs.User")
 			(effects
@@
 	(footprint "PCM_kikit:Tab"
 		(layer "F.Cu")
-		(at 92.964 56.154 90)
+		(at 92.456 56.154 90)
 		(descr "A symbol representing annotation for tab placement")
 		(property "Reference" "T4"
@@
 		)
 		(fp_text user "KIKIT: width: 3mm"
-			(at -5.5 0 360)
-			(layer "Dwgs.User")
-			(effects
+			(at -5.5 0 0)
+			(layer "Dwgs.User")
+			(effects
