File: pcb_ioexpander/project.kicad_pcb (KiCad board)
At the start: 4 copper layers, 18.3 x 25.9 mm, 47 parts, among them IC1 PCA9685PW,118, T1 Tab, T2 Tab, T3 Tab, T4 Tab

Commit message: Change ioexpander pcb
Routing:
- net +3.3V: track 8.90 -> 28.3 mm, vias 0 -> 2
- net /IO11: track 12.8 -> 9.46 mm, vias 1 -> 0
- net /IO9: track 12.0 -> 8.79 mm, vias 1 -> 0
- net /IO8: track 10.5 -> 7.37 mm, vias 1 -> 0
- net /IO6: track 6.14 -> 3.08 mm, vias 1 -> 0
- net GNDD: track 14.8 -> 12.4 mm
- net /IO10: track 11.0 -> 8.69 mm, vias 1 -> 0
- net /A2: track 19.6 -> 17.9 mm, vias 2 -> 0
- net /IO7: track 4.88 -> 3.41 mm, vias 1 -> 0
- net /A3: track 20.6 -> 19.6 mm, vias 2 -> 0
- net /A5: track 13.4 -> 14.2 mm, vias 2 -> 0
- net /A4: track 17.1 -> 16.3 mm, vias 2 -> 0
- net /A1: track 13.1 -> 12.4 mm, vias 2 -> 0
- net /IO12: track 18.0 -> 18.6 mm
- net /IO14: track 21.9 -> 22.5 mm
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- added copper zone on In2.Cu, net +3.3V
- added copper zone on F.Cu, net GNDD
- removed copper zone on F.Cu, net +3.3V
